Commit message: Major refactor for mixed integer rendezvous plans and rendezvous tracking
- Added optimal local planner from move base
- Replaced SLAM algorithm by Octomap server for faster and consistent simulations
- Added Mixed Integer Linear Program to generate rendezvous plans
- Added large scale sandbox map
- Added collision mask in robot definitions for consistent simulations
- Added modified version of ros navigation for large scale environments
- Added Rendezvous Tracking for Unknown Scenarios (RTUS) for timely rendezvous
- Added priority-based allocation policy
- Added new intermittent communication policy based on Silva2025 (ICAR)

File: src/multirobotsimulations/robots/pioneer3at/urdf/pioneer3at.urdf (robot description, URDF)
Before this commit: robot pioneer3at, 26 links, 25 joints
Links:
- link back_sonar: geometry collision mesh filename=package://multirobotsimulations/robots/pioneer3at/meshes/ba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; visual mesh filename=package://multirobotsimulations/robots/pioneer3at/meshes/ba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
- link front_sonar: geometry collision mesh filename=package://multirobotsimulations/robots/pioneer3at/meshes/fr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; visual mesh filename=package://multirobotsimulations/robots/pioneer3at/meshes/fr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
- link p3at_front_left_axle: geometry collision mesh filename=package://multirobotsimulations/robots/pioneer3at/meshes/ax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; visual mesh filename=package://multirobotsimulations/robots/pioneer3at/meshes/ax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
- link p3at_front_left_hub: geometry collision mesh filename=package://multirobotsimulations/robots/pioneer3at/meshes/le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; visual mesh filename=package://multirobotsimulations/robots/pioneer3at/meshes/le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
- link p3at_front_right_axle: geometry collision mesh filename=package://multirobotsimulations/robots/pioneer3at/meshes/ax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; visual mesh filename=package://multirobotsimulations/robots/pioneer3at/meshes/ax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
- link p3at_front_right_hub: geometry collision mesh filename=package://multirobotsimulations/robots/pioneer3at/meshes/ri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; visual mesh filename=package://multirobotsimulations/robots/pioneer3at/meshes/ri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
- link top_plate: geometry collision mesh filename=package://multirobotsimulations/robots/pioneer3at/meshes/to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; visual mesh filename=package://multirobotsimulations/robots/pioneer3at/meshes/to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
